File: hardware/board/LED_Drivers.kicad_sch (KiCad schematic)
At the start: 70 parts, among them Q901 MMBT3906, U4 TL074, U6 TL074

Commit message: update board to kicad 9
Parts:
- gave numbers to parts that had none: 54
