File: hardware/board/Output_VCA.kicad_sch (KiCad schematic)
At the start: 23 parts, among them Q801 BCM847, U2 TL074

Commit message: update board to kicad 9
Parts:
- gave numbers to parts that had none: 20
