File: hardware/board/Cutoff_CV_Driver.kicad_sch (KiCad schematic)
At the start: 19 parts, among them U2 TL074

Commit message: update board to kicad 9
Parts:
- gave numbers to parts that had none: 14

Commit message: remove test points from BOM
Parts:
- TP401: now left out of the parts list
Changed lines of the file:
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@@
 		(unit 1)
 		(exclude_from_sim no)
-		(in_bom yes)
+		(in_bom no)
 		(on_board yes)
 		(dnp no)
