File: hardware/board/Power.kicad_sch (KiCad schematic)
At the start: 39 parts, among them U1 TL074

Commit message: update board to kicad 9
Parts:
- gave numbers to parts that had none: 34

Commit message: remove test points from BOM
Parts:
- TP201, TP202, TP203: now left out of the parts list
Changed lines of the file:
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@@
 		(unit 1)
 		(exclude_from_sim no)
-		(in_bom yes)
+		(in_bom no)
 		(on_board yes)
 		(dnp no)
@@
 		(unit 1)
 		(exclude_from_sim no)
-		(in_bom yes)
+		(in_bom no)
 		(on_board yes)
 		(dnp no)
@@
 		(unit 1)
 		(exclude_from_sim no)
-		(in_bom yes)
+		(in_bom no)
 		(on_board yes)
 		(dnp no)
